File: eagle/Organ Power Supply/Organ Power Supply v0.3.sch (EAGLE design)
At the start: 22 parts, among them J1 PJ-102A, J10 CRESCENDO PEDAL, J11 POWER SWITCH, J2 USB-B, J3 54819-0519, J4 CHOIR MANUAL, J5 GREAT MANUAL, J6 SWELL MANUAL, J8 VOLUME PEDAL, J9 EXPRESSION PEDAL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

Commit message: Update eagle repos
Parts:
- removed J10: CRESCENDO PEDAL, con-molex:22-27-2031-03
- removed J11: POWER SWITCH, con-molex:22-27-2021-02
- removed J4: CHOIR MANUAL, con-molex:22-05-7038-03
- removed J5: GREAT MANUAL, con-molex:22-05-7038-03
- removed J6: SWELL MANUAL, con-molex:22-05-7038-03
- removed J7: (no value), con-molex:22-05-7058-05
- removed J8: VOLUME PEDAL, con-molex:22-27-2031-03
- removed J9: EXPRESSION PEDAL, con-molex:22-27-2031-03
- added R1: 350R, rc-master-smd:R_0805MP
- added X10: 05-JST-B5B-XH-A, con-jst-xh:05-JST-B5B-XH-A
- added X11: POWER SW, con-jst-xh:03-JST-B3B-XH-A
- added X2, X3: B2B-XH, jdc:B2B-XH
- added X4: VOLUME PEDAL, con-jst-xh:03-JST-B3B-XH-A
- added X5: EXPRESSION PEDAL, con-jst-xh:03-JST-B3B-XH-A
- added X6: CRESCENDO PEDAL, con-jst-xh:03-JST-B3B-XH-A
- added X7: CHOIR MANUAL, con-jst-xh:03-JST-B3B-XH-A
- added X8: SWELL MANUAL, con-jst-xh:03-JST-B3B-XH-A
- added X9: GREAT MANUAL, con-jst-xh:03-JST-B3B-XH-A
- C1: value 1.0uF -> 6.8uF
- C2: value 0.1uF -> 10uF
- C3: device rc-master:CP_6032-28R -> rc-master:CP_3216-18R
- U1: value AP7361 -> SPX3940
- X1: value (none) -> B2B-XH; device con-ptr500:AK500/6 -> jdc:B2B-XH
Connections:
- new net N$3: R1.1, X11-3.1
- net +3V3: now also X10-1.1, X4-1.1, X5-1.1, X6-1.1, X7-1.1, X8-1.1, X9-1.1; no longer J10-1.S, J4-1.S, J5-1.S, J6-1.S, J7-1.S, J8-1.S, J9-1.S
- net +9V: now also X1-1.1, X2-1.1, X3-1.1; no longer X1-1.KL, X1-3.KL, X1-5.KL
- net A3: now also X4-2.1; no longer J8-2.S
- net A4: now also X5-2.1; no longer J9-2.S
- net A5: now also X6-2.1; no longer J10-2.S
- net CS: now also X10-3.1; no longer J7-3.S
- net GND: now also R1.2, X1-2.1, X10-5.1, X2-2.1, X3-2.1, X4-3.1, X5-3.1, X6-3.1, X7-3.1, X8-3.1, X9-3.1; no longer J10-3.S, J4-3.S, J5-3.S, J6-3.S, J7-5.S, J8-3.S, J9-3.S, X1-2.KL, X1-4.KL, X1-6.KL
- net MISO: now also X10-2.1; no longer J7-2.S
- net N$2: now also X11-1.1; no longer J11-1.S
- net RX1: now also X7-2.1; no longer J4-2.S
- net RX2: now also X9-2.1; no longer J5-2.S
- net RX3: now also X8-2.1; no longer J6-2.S
- net SCK: now also X10-4.1; no longer J7-4.S
- net VEXT: now also X11-2.1; no longer J11-2.S
